Commit message: 修改资产库结构和关节驱动参数

File: asset/Total.SLDASM.urdf (robot description, URDF)
Before this commit: robot Total.SLDASM, 7 links, 6 joints
Links:
- link base_link: geometry collision mesh filename=meshes/base_link.STL; visual mesh filename=meshes/base_link.STL
- link left_foot: geometry collision mesh filename=meshes/left_foot.STL; visual mesh filename=meshes/left_foot.STL
- link left_leg: geometry collision mesh filename=meshes/left_leg.STL; visual mesh filename=meshes/left_leg.STL
- link left_wheel: geometry collision mesh filename=meshes/left_wheel.STL; visual mesh filename=meshes/left_wheel.STL
- link right_foot: geometry collision mesh filename=meshes/right_foot.STL; visual mesh filename=meshes/right_foot.STL
- link right_leg: geometry collision mesh filename=meshes/right_leg.STL; visual mesh filename=meshes/right_leg.STL
- link right_wheel: geometry collision mesh filename=meshes/right_wheel.STL; visual mesh filename=meshes/right_wheel.STL
